File: IRF510-Amplifier.kicad_pcb (KiCad board)
At the start: 2 copper layers, 126.4 x 81.6 mm, 55 parts, among them J1 Jack-DC, J2 BNC, J3 BNC, J4 Audio_Jack, Q1 2N3904-SMD, Q2 2SC5706, Q3 BS170F, Q4 IRF510, Q5 IRFU9024, T1 T37-43 8T:4T, T2 T37-43 25T:8T, U6 MCP1703A-2502_SOT223

Commit message: Update IRF510-Amplifier.kicad_pcb
Parts:
- moved C4 3.11 mm to (155.6, 35.2)
- moved L1 3.11 mm to (164.8, 41.9)
Routing:
- net Net-(C57-Pad1): track 19.1 -> 22.3 mm
- net +12V: track 93.0 -> 91.4 mm
Changed lines of the file:
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@@
   )
   (setup
-    (last_trace_width 1)
+    (last_trace_width 2)
     (user_trace_width 0.5)
     (user_trace_width 1)
@@
     (fp_line (start -2.54 3.825) (end 2.54 4.46) (layer F.SilkS) (width 0.127))
     (fp_circle (center 4.7625 1.92) (end 4.9869 1.92) (layer F.Fab) (width 0.4064))
-    (pad C1B thru_hole circle (at 3.81 5.73) (size 1.778 1.778) (drill 0.6) (layers *.Cu *.Mask)
+    (pad C1B thru_hole circle (at 3.81 5.73) (size 1.778 1.778) (drill 0.8) (layers *.Cu *.Mask)
       (net 21 12V-On) (solder_mask_margin 0.1016))
-    (pad C1A thru_hole circle (at -3.81 10.81) (size 1.778 1.778) (drill 0.6) (layers *.Cu *.Mask)
+    (pad C1A thru_hole circle (at -3.81 10.81) (size 1.778 1.778) (drill 0.8) (layers *.Cu *.Mask)
       (net 29 "Net-(Q1-Pad3)") (solder_mask_margin 0.1016))
-    (pad C2B thru_hole circle (at 3.81 3.19) (size 1.778 1.778) (drill 0.6) (layers *.Cu *.Mask)
+    (pad C2B thru_hole circle (at 3.81 3.19) (size 1.778 1.778) (drill 0.8) (layers *.Cu *.Mask)
       (net 26 "Net-(C13-Pad1)") (solder_mask_margin 0.1016))
-    (pad C2A thru_hole circle (at -3.81 8.27) (size 1.778 1.778) (drill 0.6) (layers *.Cu *.Mask)
+    (pad C2A thru_hole circle (at -3.81 8.27) (size 1.778 1.778) (drill 0.8) (layers *.Cu *.Mask)
       (net 1 GND) (solder_mask_margin 0.1016))
   )
@@
   )
   (module Xenir:T50_Inductor (layer F.Cu)
-    (at 165.089 45.01 270)
+    (at 164.789 41.91 270)
     (fp_text reference L1 (at 0 0.5 90) (layer F.SilkS)
       (effects (font (size 1 1) (thickness 0.15)))
@@
   )
   (module "Xenir:Capacitor 0805" (layer F.Cu)
-    (at 155.9375 38.26)
+    (at 155.6375 35.16)
     (fp_text reference C4 (at 0.5 1) (layer F.SilkS)
       (effects (font (size 0.5 0.5) (thickness 0.125)))
@@
   (segment (start 171.125 77.225) (end 169.09 75.19) (width 1) (layer F.Cu) (net 3))
   (segment (start 174.3 77.225) (end 171.125 77.225) (width 1) (layer F.Cu) (net 3))
-  (segment (start 154.3 41.2) (end 154.7 40.8) (width 1) (layer F.Cu) (net 4))
-  (segment (start 151.5 41.2) (end 154.3 41.2) (width 1) (layer F.Cu) (net 4))
+  (segment (start 154 38.1) (end 154.4 37.7) (width 1) (layer F.Cu) (net 4))
+  (segment (start 151.2 38.1) (end 154 38.1) (width 1) (layer F.Cu) (net 4))
   (segment (start 99.185 38) (end 99.318 38.133) (width 2) (layer F.Cu) (net 4))
   (segment (start 89.4 38) (end 99.185 38) (width 2) (layer F.Cu) (net 4))
@@
   (segment (start 99.318 38.133) (end 100.118 38.133) (width 2) (layer F.Cu) (net 4))
   (segment (start 100.151 38.1) (end 144.5 38.1) (width 2) (layer F.Cu) (net 4))
-  (segment (start 146.711001 40.311001) (end 144.5 38.1) (width 2) (layer F.Cu) (net 4))
-  (segment (start 150.611001 40.311001) (end 146.711001 40.311001) (width 2) (layer F.Cu) (net 4))
-  (segment (start 151.5 41.2) (end 150.611001 40.311001) (width 2) (layer F.Cu) (net 4))
+  (segment (start 144.5 38.1) (end 151.2 38.1) (width 2) (layer F.Cu) (net 4))
   (segment (start 179.52 80) (end 176.71 82.81) (width 1) (layer F.Cu) (net 5))
   (segment (start 181.35 80) (end 179.52 80) (width 1) (layer F.Cu) (net 5))
@@
   (segment (start 159.84 64.56) (end 156.5 64.56) (width 2) (layer F.Cu) (net 10))
   (segment (start 161.145 63.255) (end 159.84 64.56) (width 2) (layer F.Cu) (net 10))
-  (segment (start 161.145 49.344) (end 161.145 63.255) (width 2) (layer F.Cu) (net 10))
+  (segment (start 160.845 47.501235) (end 161.145 47.801235) (width 2) (layer F.Cu) (net 10))
+  (segment (start 161.145 47.801235) (end 161.145 63.255) (width 2) (layer F.Cu) (net 10))
+  (segment (start 160.845 46.244) (end 160.845 47.501235) (width 2) (layer F.Cu) (net 10))
   (segment (start 138.26 52.54) (end 138.3 52.5) (width 1) (layer F.Cu) (net 11))
   (segment (start 134.0375 52.54) (end 138.26 52.54) (width 1) (layer F.Cu) (net 11))
@@
     (polygon
       (pts
-        (xy 201.8 101.2) (xy 75.7 101.2) (xy 75.7 19.8) (xy 201.8 19.8)
+        (xy 201.8 101.3) (xy 75.3 101.3) (xy 75.3 19.7) (xy 201.8 19.7)
       )
     )
@@
     (polygon
       (pts
-        (xy 201.6 101.5) (xy 75.6 101.5) (xy 75.6 20.1) (xy 201.6 20.1)
+        (xy 202.1 101.3) (xy 75.8 101.3) (xy 75.8 20.1) (xy 202.1 20.1)
       )
     )

Commit message: fixed q2
Parts:
- removed C52: .1uF, Xenir:Capacitor 0805
- removed R54: 10k, Xenir:Resistor 0805
Connections:
- R52 pad 1: Net-(C52-Pad1) -> 12V-On
Routing:
- net 12V-On: track 127.6 -> 140.6 mm
- net Net-(C52-Pad1): track 8.32 -> 0.00 mm
- net Net-(Q2-Pad2): track 19.2 -> 16.4 mm
