File: IRF510-Amplifier.kicad_pcb (KiCad board)
At the start: 2 copper layers, 126.4 x 81.6 mm, 53 parts, among them J1 Jack-DC, J2 BNC, J3 BNC, J4 Audio_Jack, Q1 2N3904-SMD, Q2 2SC5706, Q3 BS170F, Q4 IRF510, Q5 IRFU9024, T1 T37-43 8T:4T, T2 T37-43 25T:8T, U6 MCP1703A-2502_SOT223

Commit message: added gerber
Parts:
- added  : , MountingHole:MountingHole_3.5mm, F.Cu at (197.5, 96.9)
- added  : , MountingHole:MountingHole_3.5mm, F.Cu at (197.3, 24.4)
- added  : , MountingHole:MountingHole_3.5mm, F.Cu at (80.2, 96.8)
- added  : , MountingHole:MountingHole_3.5mm, F.Cu at (80.1, 24.3)
Other:
- board text added: "IRF510 Amplifier"
- board text removed: "10W Amplifier"
Changed lines of the file:
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@@
     (tracks 170)
     (zones 0)
-    (modules 53)
+    (modules 57)
     (nets 29)
   )
@@
     (add_net "Net-(RV1-Pad1)")
   )
+  (module MountingHole:MountingHole_3.5mm (layer F.Cu)
+    (at 197.5 96.9)
+    (descr "Mounting Hole 3.5mm, no annular")
+    (tags "mounting hole 3.5mm no annular")
+    (attr virtual)
+    (fp_text reference " " (at 0 -4.5) (layer F.SilkS)
+      (effects (font (size 1 1) (thickness 0.15)))
+    )
+    (fp_text value " " (at 0 4.5) (layer F.Fab)
+      (effects (font (size 1 1) (thickness 0.15)))
+    )
+    (fp_text user %R (at 0.3 0) (layer F.Fab)
+      (effects (font (size 1 1) (thickness 0.15)))
+    )
+    (fp_circle (center 0 0) (end 3.5 0) (layer Cmts.User) (width 0.15))
+    (fp_circle (center 0 0) (end 3.75 0) (layer F.CrtYd) (width 0.05))
+    (pad 1 np_thru_hole circle (at 0 0) (size 3.5 3.5) (drill 3.5) (layers *.Cu *.Mask))
+  )
+  (module MountingHole:MountingHole_3.5mm (layer F.Cu)
+    (at 197.3 24.4)
+    (descr "Mounting Hole 3.5mm, no annular")
+    (tags "mounting hole 3.5mm no annular")
+    (attr virtual)
+    (fp_text reference " " (at 0 -4.5) (layer F.SilkS)
+      (effects (font (size 1 1) (thickness 0.15)))
+    )
+    (fp_text value " " (at 0 4.5) (layer F.Fab)
+      (effects (font (size 1 1) (thickness 0.15)))
+    )
+    (fp_circle (center 0 0) (end 3.75 0) (layer F.CrtYd) (width 0.05))
+    (fp_circle (center 0 0) (end 3.5 0) (layer Cmts.User) (width 0.15))
+    (fp_text user %R (at 0.3 0) (layer F.Fab)
+      (effects (font (size 1 1) (thickness 0.15)))
+    )
+    (pad 1 np_thru_hole circle (at 0 0) (size 3.5 3.5) (drill 3.5) (layers *.Cu *.Mask))
+  )
+  (module MountingHole:MountingHole_3.5mm (layer F.Cu)
+    (at 80.2 96.8)
+    (descr "Mounting Hole 3.5mm, no annular")
+    (tags "mounting hole 3.5mm no annular")
+    (attr virtual)
+    (fp_text reference " " (at 0 -4.5) (layer F.SilkS)
+      (effects (font (size 1 1) (thickness 0.15)))
+    )
+    (fp_text value " " (at 0 4.5) (layer F.Fab)
+      (effects (font (size 1 1) (thickness 0.15)))
+    )
+    (fp_text user %R (at 0.3 0) (layer F.Fab)
+      (effects (font (size 1 1) (thickness 0.15)))
+    )
+    (fp_circle (center 0 0) (end 3.5 0) (layer Cmts.User) (width 0.15))
+    (fp_circle (center 0 0) (end 3.75 0) (layer F.CrtYd) (width 0.05))
+    (pad 1 np_thru_hole circle (at 0 0) (size 3.5 3.5) (drill 3.5) (layers *.Cu *.Mask))
+  )
+  (module MountingHole:MountingHole_3.5mm (layer F.Cu)
+    (at 80.1 24.3)
+    (descr "Mounting Hole 3.5mm, no annular")
+    (tags "mounting hole 3.5mm no annular")
+    (attr virtual)
+    (fp_text reference " " (at 0 -4.5) (layer F.SilkS)
+      (effects (font (size 1 1) (thickness 0.15)))
+    )
+    (fp_text value " " (at 0 4.5) (layer F.Fab)
+      (effects (font (size 1 1) (thickness 0.15)))
+    )
+    (fp_circle (center 0 0) (end 3.75 0) (layer F.CrtYd) (width 0.05))
+    (fp_circle (center 0 0) (end 3.5 0) (layer Cmts.User) (width 0.15))
+    (fp_text user %R (at 0.3 0) (layer F.Fab)
+      (effects (font (size 1 1) (thickness 0.15)))
+    )
+    (pad 1 np_thru_hole circle (at 0 0) (size 3.5 3.5) (drill 3.5) (layers *.Cu *.Mask))
+  )
   (module "Xenir:Capacitor 0805" (layer F.Cu)
     (at 111.9625 51.16)
@@
       (net 2 "Net-(C3-Pad1)"))
   )
-  (gr_text "10W Amplifier" (at 170 29.7) (layer F.SilkS)
+  (gr_text "IRF510 Amplifier" (at 168.1 28.4) (layer F.SilkS)
     (effects (font (size 4 4) (thickness 0.5)))
   )
