File: IRF510-Amplifier.sch (KiCad schematic (older format))
At the start: 55 parts, among them J1 Jack-DC, J2 BNC, J3 BNC, J4 Audio_Jack, Q1 2N3904-SMD, Q2 2SC5706, Q3 BS170F, Q4 IRF510, Q5 IRFU9024, T1 T37-43 8T:4T, T2 T37-43 25T:8T, U6 MCP1703A-2502_SOT223

Commit message: fixed q2
Parts:
- removed C52: .1uF, Xenir:Capacitor 0805, symbol Xenir:Capacitor
- removed R54: 10k, Xenir:Resistor 0805, symbol Xenir:Resistor
Connections:
- net 12V-On: now also R52.1
Changed lines of the file:
@@
 	1    0    0    -1
 $EndComp
-$Comp
-L Xenir:Resistor R54
-U 1 1 5F4BFB3E
-P 4250 3350
-F 0 "R54" H 4250 3425 28  0000 C CNN
-F 1 "10k" H 4250 3275 28  0000 C CNN
-F 2 "Xenir:Resistor 0805" H 4250 3250 50  0001 C CNN
-F 3 "" H 4250 3250 50  0001 C CNN
-	1    4250 3350
-	-1   0    0    1
-$EndComp
-Wire Wire Line
-	4050 3700 4050 3650
-$Comp
-L Xenir:Capacitor C52
-U 1 1 5F4C0F3A
-P 4300 3650
-F 0 "C52" H 4300 3775 28  0000 C CNN
-F 1 ".1uF" H 4300 3525 28  0000 C CNN
-F 2 "Xenir:Capacitor 0805" H 4300 3500 50  0001 C CNN
-F 3 "" H 4300 3500 50  0001 C CNN
-	1    4300 3650
-	1    0    0    -1
-$EndComp
-Wire Wire Line
-	4150 3650 4050 3650
-Connection ~ 4050 3650
 Wire Wire Line
 	4050 4100 4350 4100
-Wire Wire Line
-	4450 3650 4650 3650
-Wire Wire Line
-	4650 3650 4650 3900
-Connection ~ 4650 3650
 $Comp
 L Xenir:Capacitor C53
@@
 Connection ~ 10350 2750
 Wire Wire Line
-	4450 3350 4650 3350
-Wire Wire Line
-	4650 3350 4650 3650
-Wire Wire Line
-	4050 3350 4050 3650
-Wire Wire Line
 	4050 4350 4050 4100
 $Comp
@@
 	1    0    0    -1
 $EndComp
-Connection ~ 4650 3350
 $Comp
 L Device:R_POT RV1
@@
 	1    0    0    -1
 $EndComp
+Wire Wire Line
+	4650 3350 4650 3900
+Wire Wire Line
+	4050 3350 4050 3700
+Text GLabel 4050 3350 1    50   Input ~ 0
+12V-On
 $EndSCHEMATC
