File: IRF510-Amplifier.sch (KiCad schematic (older format))
At the start: 53 parts, among them J1 Jack-DC, J2 BNC, J3 BNC, J4 Audio_Jack, Q1 2N3904-SMD, Q2 2SC5706, Q3 BS170F, Q4 IRF510, Q5 IRFU9024, T1 T37-43 8T:4T, T2 T37-43 25T:8T, U6 MCP1703A-2502_SOT223

Commit message: dd
Parts:
- R8: value 1k -> 100
Other:
- note added: "C3"
- note added: "C5"
- note added: "C7"
- note added: "C8"
- note added: "L3"
- note added: "L4"

Commit message: gg
Parts:
- R64: value 4.7k -> 24k
- R65: value 1k -> 6.8k
Changed lines of the file:
@@
 P 1800 3700
 F 0 "R64" H 1800 3775 28  0000 C CNN
-F 1 "4.7k" H 1800 3625 28  0000 C CNN
+F 1 "24k" H 1800 3625 28  0000 C CNN
 F 2 "Xenir:Resistor 0805" H 1800 3600 50  0001 C CNN
 F 3 "" H 1800 3600 50  0001 C CNN
@@
 P 1800 4400
 F 0 "R65" H 1800 4475 28  0000 C CNN
-F 1 "1k" H 1800 4325 28  0000 C CNN
+F 1 "6.8k" H 1800 4325 28  0000 C CNN
 F 2 "Xenir:Resistor 0805" H 1800 4300 50  0001 C CNN
 F 3 "" H 1800 4300 50  0001 C CNN
